File: PCBs/signal_processing/signal_processing.sch (KiCad schematic (older format))
At the start: 140 parts, among them IC1 AD8066, IC2 ADG701BRTZN, IC3 AD8066, IC4 AD8066, IC5 LT1713, IC6 LT1713, IC7 AD8066, X1 87437-0443, X2 87437-0443, X3 87437-0443

Commit message: Reorganization of pcb files
Parts:
- removed A1, A2, A3: SMA-EDGE-0.062, signal_processing:CONSMA003.062, symbol signal_processing-eagle-import:LINX-SMA-EDGE-0.062
- removed C10, C14, C50: 100n/50V, signal_processing:C0603, symbol signal_processing-eagle-import:C-EUC0603
- removed C12, C16: 47u/6V, signal_processing:SMC_B, symbol signal_processing-eagle-import:CPOL-EUSMCB
- removed C5: 1n/100V, signal_processing:C0603, symbol signal_processing-eagle-import:C-EUC0603
- removed C52: 4,7u/6V, signal_processing:SMC_A, symbol signal_processing-eagle-import:CPOL-EUSMCA
- removed C7: 4,7u/50V, signal_processing:C1206, symbol signal_processing-eagle-import:C-EUC1206
- removed LED2, LED4, LED6: GREEN, signal_processing:CHIPLED_0603, symbol signal_processing-eagle-import:LEDCHIPLED_0603
- removed R12, R17: 300, signal_processing:R0603, symbol signal_processing-eagle-import:R-EU_R0603
- removed R2: 43k, signal_processing:R0603, symbol signal_processing-eagle-import:R-EU_R0603
- removed R20, R21, R23, R24, R28, R29, R32, R33, R36, R40, R41, R44, R45: 1, signal_processing:R0603, symbol signal_processing-eagle-import:R-EU_R0603
- removed X1, X2, X3: 87437-0443, signal_processing:87437-0443, symbol signal_processing-eagle-import:87438-0487437-0443
- added C5: 100n/50V, Capacitor_SMD:C_0603_1608Metric, symbol Device:C
- added C7: 4,7u/6V, Capacitor_Tantalum_SMD:CP_EIA-3216-18_Kemet-A, symbol Device:CP
- added J1, J2, J6: 874380443, semiconductor_radiation_detector:87438-0443, symbol semiconductor_radiation_detector:874380443
- added J3, J4, J5: CON-SMA-EDGE-S, semiconductor_radiation_detector:CON-SMA-EDGE-S, symbol semiconductor_radiation_detector:CON-SMA-EDGE-S
- added L1, L10, L11, L12, L13, L2, L3, L4, L5, L6, L7, L8, L9: 1u, Inductor_SMD:L_0603_1608Metric, symbol Device:L
- added RV1: 500, Potentiometer_SMD:Potentiometer_Bourns_3224W_Vertical, symbol Device:R_POT
- added RV2: 10, Potentiometer_SMD:Potentiometer_Bourns_3224W_Vertical, symbol Device:R_POT
- C1, C13, C17, C18, C2, C21, C22, C25, C26, C27, C28, C29, C3, C32, C33, C36, C38, C39, C4, C40, C41, C44, C45, C46, C47, C51, C54, C55, C8, C9: footprint signal_processing:C0603 -> Capacitor_SMD:C_0603_1608Metric; symbol signal_processing-eagle-import:C-EUC0603 -> Device:C
- C11, C15: footprint signal_processing:SMC_B -> Capacitor_Tantalum_SMD:CP_EIA-3528-21_Kemet-B; symbol signal_processing-eagle-import:CPOL-EUSMCB -> Device:CP
- C19, C20, C23, C24, C30, C31, C34, C35, C37, C42, C43, C48, C49, C53: footprint signal_processing:SMC_A -> Capacitor_Tantalum_SMD:CP_EIA-3216-18_Kemet-A; symbol signal_processing-eagle-import:CPOL-EUSMCA -> Device:CP
- C6: footprint signal_processing:C1206 -> Capacitor_SMD:C_1206_3216Metric; symbol signal_processing-eagle-import:C-EUC1206 -> Device:C
- D1, D2, D3, D4, D5, D6, D7: footprint signal_processing:SOD2514X100N -> Diode_SMD:D_SOD-323; symbol signal_processing-eagle-import:BAS140 -> Device:D_Schottky
- IC1, IC3, IC4, IC7: footprint signal_processing:MSOP8 -> Package_SO:MSOP-8_3x3mm_P0.65mm; symbol signal_processing-eagle-import:AD8066 -> semiconductor_radiation_detector:AD8066
- IC2: footprint signal_processing:SOT23-6 -> Package_TO_SOT_SMD:SOT-23-6; symbol signal_processing-eagle-import:ADG701BRTZN -> semiconductor_radiation_detector:ADG701
- IC5, IC6: footprint signal_processing:MSOP8 -> Package_SO:MSOP-8_3x3mm_P0.65mm; symbol signal_processing-eagle-import:LT1713 -> semiconductor_radiation_detector:LT1713
- LED1, LED3, LED5: footprint signal_processing:CHIPLED_0603 -> LED_SMD:LED_0603_1608Metric; symbol signal_processing-eagle-import:LEDCHIPLED_0603 -> Device:LED
- R1, R10, R11, R13, R14, R15, R16, R18, R19, R22, R25, R26, R27, R3, R30, R31, R34, R35, R37, R38, R39, R4, R42, R43, R46, R47, R48, R49, R5, R50, R51, R52, R53, R54, R55, R56, R57, R58, R59, R6, R7, R8, R9: footprint signal_processing:R0603 -> Resistor_SMD:R_0603_1608Metric; symbol signal_processing-eagle-import:R-EU_R0603 -> Device:R
- U1: renamed from IC2; value ADG701BRTZN -> ADG701; footprint signal_processing:SOT23-6 -> Package_TO_SOT_SMD:SOT-23-6; symbol signal_processing-eagle-import:ADG701BRTZN -> semiconductor_radiation_detector:ADG701
Connections:
- wire segments 423 -> 403
Other:
- note added: "Power supply filtering and fowarding"
- note removed: "Common resistors \nor ferrite beads"
- note removed: "Power supply connector and fowarding"

Commit message: finished preamplifier board redesigning
Parts:
- added R44, R46: 1k, Resistor_SMD:R_0603_1608Metric, symbol Device:R
- added R45, R47: 2k, Resistor_SMD:R_0603_1608Metric, symbol Device:R
- IC5: renamed from IC2; value ADG701BRTZN -> ADG701
- renumbered C15 to C10, C17 to C11, C18 to C12, C19 to C13, C20 to C14, C21 to C15, C22 to C16, C23 to C17, C24 to C18, C26 to C19, C25 to C20, C29 to C21, C27 to C22, C28 to C23, C30 to C24, C31 to C25, C32 to C26, C33 to C27, C34 to C28, C35 to C29, C36 to C30, C37 to C31, C38 to C32, C39 to C33, C40 to C34, C41 to C35, C42 to C36, C43 to C37, C44 to C38, C45 to C39, C46 to C40, C47 to C41, C48 to C42, C49 to C43, C51 to C44, C5 to C45, C53 to C46, C7 to C47, C54 to C48, C55 to C49, C6 to C5, C8 to C6, C9 to C7, C11 to C8, C13 to C9, IC3 to IC1, IC7 to IC1, IC3 to IC2, IC7 to IC2, IC1 to IC2, IC4 to IC3, IC1 to IC3, IC3 to IC4, IC7 to IC4, IC5 to IC7, LED3 to LED2, LED5 to LED3, R3 to R1, R13 to R10, R14 to R12, R15 to R13, R18 to R14, R16 to R15, R19 to R16, R22 to R17, R25 to R18, R26 to R19, R4 to R2, R27 to R20, R30 to R21, R31 to R22, R34 to R23, R35 to R24, R37 to R25, R38 to R26, R39 to R27, R42 to R28, R43 to R29, R5 to R3, R49 to R30, R50 to R31, R46 to R32, R47 to R33, R48 to R34, R51 to R35, R52 to R36, R55 to R37, R53 to R38, R54 to R39, R1 to R4, R56 to R40, R57 to R41, R58 to R42, R59 to R43, R6 to R5, R7 to R6, R8 to R7, R9 to R8, R10 to R9
Connections:
- wire segments 403 -> 413
Other:
- note added: "Power supply filtering and forwarding"
- note removed: "Power supply filtering and fowarding"

Commit message: sp board update
Parts:
- added C50: 1p/50V, Capacitor_SMD:C_0603_1608Metric, symbol Device:C
- C33: renamed from C21; value 200p/50V -> 2,2n/50V
- C34: renamed from C38; value 180p/50V -> 2,2n/50V
- C35: renamed from C49; value 160p/50V -> 2,2n/50V
- C36: renamed from C20; value 200p/50V -> 2,2n/50V
- C37: renamed from C35; value 180p/50V -> 2,2n/50V
- C38: renamed from C48; value 160p/50V -> 220p/50V
- R10: renamed from R20; value 9,1k -> 820
- R11: renamed from R29; value 8,2k -> 1k
- R12: renamed from R43; value 6,8k -> 680
- R13: renamed from R18; value 1,8k -> 270
- R14: renamed from R27; value 2k -> 270
- R15: renamed from R40; value 3,3k -> 470
- R4: renamed from R16; value 3k -> 390
- R5: renamed from R17; value 33k -> 2,4k
- R6: renamed from R23; value 3,6k -> 330
- R7: renamed from R25; value 30k -> 3,3k
- R8: renamed from R32; value 6,2k -> 560
- renumbered C4 to C1, C17 to C10, C22 to C11, C24 to C12, C26 to C13, C28 to C14, C33 to C15, C36 to C16, C40 to C17, C42 to C18, C30 to C19, C5 to C2, C31 to C20, C12 to C21, C14 to C22, C16 to C23, C18 to C24, C23 to C25, C25 to C26, C29 to C28, C34 to C29, C7 to C3, C37 to C30, C41 to C31, C43 to C32, C3 to C39, C8 to C4, C19 to C40, C45 to C41, C47 to C42, C1 to C43, C2 to C44, C39 to C45, C32 to C46, C6 to C47, C44 to C48, C46 to C49, C9 to C5, C10 to C6, C11 to C7, C13 to C8, C15 to C9, D7 to D1, D5 to D2, D6 to D3, D1 to D5, D2 to D6, D3 to D7, IC4 to IC1, IC2 to IC1, IC1 to IC2, IC4 to IC2, IC2 to IC4, IC1 to IC4, U1 to IC5, IC7 to IC6, IC6 to IC7, J3 to J1, J1 to J2, J2 to J3, J6 to J4, J4 to J5, J5 to J6, L6 to L10, L8 to L11, L11 to L12, L3 to L2, L5 to L3, L7 to L4, L10 to L5, L12 to L6, L9 to L7, L2 to L8, L4 to L9, LED3 to LED1, LED1 to LED2, LED2 to LED3, R4 to R1, R6 to R16, R1 to R17, R33 to R18, R13 to R19, R11 to R2, R14 to R20, R22 to R21, R3 to R22, R7 to R23, R38 to R24, R42 to R25, R19 to R26, R10 to R27, R34 to R28, R39 to R29, R15 to R3, R44 to R30, R12 to R31, R21 to R32, R45 to R33, R28 to R34, R24 to R35, R2 to R36, R26 to R38, R30 to R39, R5 to R40, R46 to R41, R36 to R42, R41 to R43, R47 to R44, R31 to R45, R8 to R46, R9 to R47, R35 to R9, RV2 to RV1, RV1 to RV2
Connections:
- wire segments 413 -> 417
